File: hardware/deskclock2/deskclock2.kicad_pcb (KiCad board)
At the start: 2 copper layers, 86.4 x 99.1 mm, 29 parts, among them J1 TEMP SENSOR, J2 IR RECEIVER, J3 DIGITAL, J4 SERIAL, J5 3.3V POWER, J6 ANALOG, J7 5V POWER, J8 TOUCH LCD, SW1 SW_Push, SW2 SW_Push, SW3 SW_Push, SW4 SW_Push, SW5 SW_Push, SW6 SW_Push, SW7 SW_Push, SW8 SW_Push, SW9 Flash, U1 Adfruit_LCD_Breakout_Touch, U3 MCP23008

Commit message: Revision 1 complete
Parts:
- moved U1 5.30 mm to (135.9, 91.4)
- moved J8 1.27 mm to (128.3, 81.3)
Routing:
- net T_IRQ: track 58.8 -> 60.1 mm
- net LCD_POCI: track 39.3 -> 40.6 mm
- net +5V: track 112.1 -> 113.4 mm
- net LCD_SCK: track 51.3 -> 52.5 mm
- net LCD_PICO: track 41.0 -> 42.3 mm
- net LCD_CS: track 25.3 -> 25.8 mm
- net SDA: track 62.4 -> 62.9 mm
- net SCL: track 67.1 -> 67.6 mm
- net LCD_DC: track 31.8 -> 32.4 mm
- net GND: vias 8 -> 9
Other:
- board text added: "3.3V"
- board text added: "5V"
- board text added: "A0"
- board text added: "A1"
- board text added: "A2"
- board text added: "A3"
- board text added: "A4"
- board text added: "A5"
- board text added: "CS"
- board text added: "D/C"
- board text added: "D11"
- board text added: "D12"
- board text added: "D13"
- board text added: "DeskClock2 Rev. 1"
- board text added: "GND"
- board text added: "PICO (MOSI)"
- board text added: "POCI (MISO)"
- board text added: "RX"
- board text added: "SCK"
- board text added: "TX"
- board text added: "T_IRQ"
- board text added: "T_SCL"
- board text added: "T_SDA"
