File: hardware/deskclock2/deskclock2.kicad_sch (KiCad schematic)
At the start: 29 parts, among them J1 TEMP SENSOR, J2 IR RECEIVER, J3 DIGITAL, J4 SERIAL, J5 3.3V POWER, J6 ANALOG, J7 5V POWER, J8 TOUCH LCD, SW1 SW_Push, SW2 SW_Push, SW3 SW_Push, SW4 SW_Push, SW5 SW_Push, SW6 SW_Push, SW7 SW_Push, SW8 SW_Push, SW9 Flash, U1 Adfruit_LCD_Breakout_Touch, U3 MCP23008

Commit message: Revision 1 complete
Other:
- title: (none) -> Deskclock2
Changed lines of the file:
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@@
 (kicad_sch (version 20211123) (generator eeschema)
   (paper "A4")
+  (title_block
+    (title "Deskclock2")
+    (rev "1")
+  )
   (junction (at 74.93 121.92) (diameter 0) (color 0 0 0 0)
   )
