File: hardware/DeskClock2/DeskClock2.kicad_sch (KiCad schematic)
At the start: 29 parts, among them J1 TEMP SENSOR, J2 IR RECEIVER, J3 DIGITAL, J4 SERIAL, J5 3.3V POWER, J6 ANALOG, J7 5V POWER, J8 TOUCH LCD, SW1 SW_Push, SW2 SW_Push, SW3 SW_Push, SW4 SW_Push, SW5 SW_Push, SW6 SW_Push, SW7 SW_Push, SW8 SW_Push, SW9 Flash, U1 Adfruit_LCD_Breakout_Touch, U3 MCP23008

Commit message: Changed capitalization of file names in hardware/
Other:
- title: Deskclock2 -> DeskClock2
Changed lines of the file:
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@@
   (paper "A4")
   (title_block
-    (title "Deskclock2")
+    (title "DeskClock2")
     (rev "1")
   )
